Commit message: Updates getting this project going.

File: ur_description/urdf/ur10.urdf.xacro (robot description, xacro)
@@ -319,5 +319,5 @@
     <joint name="camera_joint" type="fixed">
     <axis xyz="0 1 0" />
-    <origin xyz="-0.0 0.055 0" rpy="0 0 0"/>
+    <origin xyz="-0.02 0.055 0" rpy="0 0 0"/>
     <parent link="ee_link"/>
     <child link="camera_link"/>
